File: dev_board.kicad_pcb (KiCad board)
At the start: 6 copper layers, 109 x 115 mm, 225 parts, among them J1 Conn_02x13_Odd_Even, J2 Conn_02x13_Odd_Even, J4 Jack, J5 Conn_01x06, J7 Jack, J9 Barrel_Jack, Q1 STR2P3LLH6(Pfet), Q10 MMBT3904, Q2 2N3904, Q3 MMBT3904, Q4 IPD60R145, Q5 IRLML0060TRPBF, Q6 IPD60R145, Q9 MMBT3904, SW1 SW_SPST, SW10 LAUNCH, SW3 ARM, U1 LT3420, U10 AMC3330, U11 AT25xxx, U12 TLV74318, U13 LM809, U14 AMC3302, U17 AD7352, U18 IR2127, U2 TLV74318, U23 TLV74325, U3 AD7352, U4 TLV74325, U5 LMO78_03-1.0, U6 4945, U7 MCP1416, U8 AMC3330, X1 ASE-48MHz

Commit message: Closer to tapeout, Digikey BOM added
Connections:
- J1 pad 3: +1V1 -> unconnected-(J1-Pin_3-Pad3)
Routing:
- net +1V1: track 45.2 -> 19.7 mm
- net GND: vias 81 -> 76
- net +3.3V: vias 33 -> 32
- added copper zone on In3.Cu, net GND
- added copper zone on In4.Cu, net GND
- removed copper zone on In3.Cu, net +1V1
- removed copper zone on In4.Cu, net +3.3V
Other:
- board size 109 x 115 mm -> 109 x 114.5 mm

Commit message: Tapeout v01.2
Parts:
- added C100: 0.1u, Capacitor_SMD:C_0603_1608Metric, B.Cu at (192.3, 117.1)
- added C101: 0.1u, Capacitor_SMD:C_0603_1608Metric, B.Cu at (176.8, 117.1)
- added C102: 0.1u, Capacitor_SMD:C_0603_1608Metric, B.Cu at (164.8, 139.4)
- added C103: 0.1u, Capacitor_SMD:C_0603_1608Metric, B.Cu at (180.1, 117.1)
- added C104: 1u, Capacitor_SMD:C_0603_1608Metric, B.Cu at (164.8, 117.9)
- added C105: 0.1u, Capacitor_SMD:C_0603_1608Metric, B.Cu at (186.2, 117.1)
- added C106: 0.1u, Capacitor_SMD:C_0603_1608Metric, B.Cu at (195.7, 142.2)
- added C108: 0.1u, Capacitor_SMD:C_0603_1608Metric, B.Cu at (192.3, 133.5)
- added C109: 0.1u, Capacitor_SMD:C_0603_1608Metric, B.Cu at (185.9, 143.0)
- added C110: 0.1u, Capacitor_SMD:C_0603_1608Metric, B.Cu at (166.5, 142.4)
- added C115: 1u, Capacitor_SMD:C_0603_1608Metric, F.Cu at (175.5, 137.2)
- added C116: 0.1u, Capacitor_SMD:C_0603_1608Metric, B.Cu at (164.8, 127.0)
- added C119: 0.1u, Capacitor_SMD:C_0603_1608Metric, F.Cu at (183.4, 125.0)
- added C120: 0.1u, Capacitor_SMD:C_0603_1608Metric, B.Cu at (168.9, 142.2)
- added C121: 0.1u, Capacitor_SMD:C_0603_1608Metric, B.Cu at (164.8, 124.0)
- added C122: 0.1u, Capacitor_SMD:C_0603_1608Metric, B.Cu at (173.5, 117.1)
- added C123: 0.1u, Capacitor_SMD:C_0603_1608Metric, B.Cu at (170.2, 117.1)
- added C124: 0.1u, Capacitor_SMD:C_0603_1608Metric, B.Cu at (182.9, 117.1)
- added C125: 1u, Capacitor_SMD:C_0603_1608Metric, F.Cu at (198.1, 128.0)
- added C126: 1u, Capacitor_SMD:C_0603_1608Metric, B.Cu at (194.8, 130.6)
- added C127: 0.1u, Capacitor_SMD:C_0603_1608Metric, F.Cu at (192.3, 128.0)
- added C130: 0.1u, Capacitor_SMD:C_0603_1608Metric, B.Cu at (192.5, 129.8)
- added C131: 0.1u, Capacitor_SMD:C_0603_1608Metric, F.Cu at (190.0, 128.0)
- added C139: 0.1u, Capacitor_SMD:C_0603_1608Metric, B.Cu at (190.0, 130.3)
- added C140: 0.1u, Capacitor_SMD:C_0603_1608Metric, B.Cu at (190.8, 135.6)
- added C141: 1u, Capacitor_SMD:C_0603_1608Metric, B.Cu at (180.8, 142.2)
- added C142: 0.1u, Capacitor_SMD:C_0603_1608Metric, B.Cu at (180.6, 143.8)
- added C143: 0.1u, Capacitor_SMD:C_0603_1608Metric, B.Cu at (175.5, 142.2)
- added C144: 0.1u, Capacitor_SMD:C_0603_1608Metric, B.Cu at (172.5, 142.2)
- added C51: 4.7u, Capacitor_SMD:C_1206_3216Metric, B.Cu at (196.3, 117.6)
- added C52: 4.7u, Capacitor_SMD:C_1206_3216Metric, B.Cu at (195.6, 144.3)
- added C58: 4.7u, Capacitor_SMD:C_1206_3216Metric, B.Cu at (196.6, 133.9)
- added C90: 0.1u, Capacitor_SMD:C_0603_1608Metric, B.Cu at (183.1, 143.0)
- added C91: 1u, Capacitor_SMD:C_0603_1608Metric, B.Cu at (164.8, 136.4)
- added C92: 0.1u, Capacitor_SMD:C_0603_1608Metric, B.Cu at (167.1, 117.1)
- added C93: 0.1u, Capacitor_SMD:C_0603_1608Metric, B.Cu at (190.0, 133.2)
- added C94: 0.1u, Capacitor_SMD:C_0603_1608Metric, B.Cu at (189.7, 141.2)
- added C96: 0.1u, Capacitor_SMD:C_0603_1608Metric, B.Cu at (189.2, 117.1)
- added C97: 0.1u, Capacitor_SMD:C_0603_1608Metric, B.Cu at (191.4, 141.2)
- added C98: 1u, Capacitor_SMD:C_0603_1608Metric, B.Cu at (188.2, 141.2)
- added C99: 0.1u, Capacitor_SMD:C_0603_1608Metric, B.Cu at (196.6, 135.9)
- added D10: Yel, LED_SMD:LED_0603_1608Metric, F.Cu at (171.4, 116.8)
- added D11: Yel, LED_SMD:LED_0603_1608Metric, F.Cu at (174.6, 116.8)
- added D12: Yel, LED_SMD:LED_0603_1608Metric, F.Cu at (177.8, 116.8)
- added D13: Yel, LED_SMD:LED_0603_1608Metric, F.Cu at (181.0, 116.8)
- added D14: Yel, LED_SMD:LED_0603_1608Metric, F.Cu at (184.2, 116.8)
- added D15: Yel, LED_SMD:LED_0603_1608Metric, F.Cu at (187.1, 116.8)
- added D16: BAV99, Package_TO_SOT_SMD:SOT-23, F.Cu at (186.7, 121.2)
- added D3: Yel, LED_SMD:LED_0603_1608Metric, F.Cu at (165.7, 116.8)
- added D8: Yel, LED_SMD:LED_0603_1608Metric, F.Cu at (168.5, 116.8)
- added FB2: Ferrite, Inductor_SMD:L_0603_1608Metric, B.Cu at (192.3, 118.5)
- added FB3: Ferrite, Inductor_SMD:L_0603_1608Metric, B.Cu at (164.8, 120.9)
- added FB4: Ferrite, Inductor_SMD:L_0603_1608Metric, B.Cu at (164.8, 142.5)
- added FB8: Ferrite, Inductor_SMD:L_0603_1608Metric, B.Cu at (190.0, 137.9)
- added J10: Conn_02x05_Odd_Even, Connector_PinHeader_2.54mm:PinHeader_2x05_P2.54mm_Vertical_SMD, F.Cu at (169.2, 129.0)
- added J12: HDMI_D_1.4, Connector_HDMI:HDMI_A_Amphenol_10029449-x01xLF_Horizontal, F.Cu at (196.0, 139.0)
- added J14: Conn_02x05_Odd_Even, Connector_PinHeader_2.54mm:PinHeader_2x05_P2.54mm_Vertical_SMD, F.Cu at (182.6, 141.7)
- added J3: Conn_02x13_Odd_Even, Connector_PinSocket_2.54mm:PinSocket_2x13_P2.54mm_Vertical, B.Cu at (196.8, 149.9)
- added J6: Conn_02x13_Odd_Even, Connector_PinSocket_2.54mm:PinSocket_2x13_P2.54mm_Vertical, B.Cu at (196.8, 111.8)
- added LS2: Speaker, Buzzer_Beeper:PUIAudio_SMT_0825_S_4_R, F.Cu at (194.3, 121.4)
- added Q7: MMBT3904, Package_TO_SOT_SMD:SOT-23, B.Cu at (165.9, 145.8)
- added R101: 10K, Resistor_SMD:R_0603_1608Metric, B.Cu at (176.3, 144.5)
- added R56: 0R, Resistor_SMD:R_0603_1608Metric, B.Cu at (177.0, 147.1)
- added R57: 1K, Resistor_SMD:R_0603_1608Metric, F.Cu at (165.7, 118.1)
- added R58: 1K, Resistor_SMD:R_0603_1608Metric, F.Cu at (168.5, 118.1)
- added R59: 1K, Resistor_SMD:R_0603_1608Metric, F.Cu at (171.4, 118.1)
- added R60: 1K, Resistor_SMD:R_0603_1608Metric, F.Cu at (174.6, 118.1)
- added R65: 1K, Resistor_SMD:R_0603_1608Metric, F.Cu at (177.8, 118.1)
- added R66: 1K, Resistor_SMD:R_0603_1608Metric, F.Cu at (181.0, 118.1)
- added R71: 1K, Resistor_SMD:R_0603_1608Metric, F.Cu at (184.2, 118.1)
- added R72: 1K, Resistor_SMD:R_0603_1608Metric, F.Cu at (187.1, 118.1)
- added R73: 1K, Resistor_SMD:R_0603_1608Metric, B.Cu at (168.9, 143.8)
- added R74: 10K, Resistor_SMD:R_0603_1608Metric, F.Cu at (181.2, 121.4)
- added R75: 10K, Resistor_SMD:R_0603_1608Metric, F.Cu at (172.1, 121.4)
- added R76: 10K, Resistor_SMD:R_0603_1608Metric, F.Cu at (168.9, 121.4)
- added R77: 1K, Resistor_SMD:R_0603_1608Metric, F.Cu at (175.3, 121.4)
- added R78: 10K, Resistor_SMD:R_0603_1608Metric, F.Cu at (165.7, 121.3)
- added R84: 0R, Resistor_SMD:R_0603_1608Metric, B.Cu at (164.8, 130.2)
- added R86: 22R, Resistor_SMD:R_0603_1608Metric, F.Cu at (186.9, 125.2)
- added R87: 22R, Resistor_SMD:R_0603_1608Metric, B.Cu at (172.7, 146.3)
- added R88: DNI, Resistor_SMD:R_0603_1608Metric, B.Cu at (174.5, 146.3)
- added R90: 0R, Resistor_SMD:R_0603_1608Metric, B.Cu at (180.6, 145.3)
- added R91: 22R, Resistor_SMD:R_0603_1608Metric, F.Cu at (178.3, 121.4)
- added R97: 0R, Resistor_SMD:R_0603_1608Metric, B.Cu at (183.6, 145.3)
- added SW12: SW_DIP_x03, Button_Switch_SMD:SW_DIP_SPSTx03_Slide_Omron_A6S-310x_W8.9mm_P2.54mm, F.Cu at (169.2, 142.2)
- added SW2: LAUNCH, myspace pcb:SW_SPST_HP03, F.Cu at (177.5, 129.0)
- added TP10: ~, TestPoint:TestPoint_Pad_D1.0mm, B.Cu at (178.1, 142.2)
- added TP11: ~, TestPoint:TestPoint_Pad_D1.0mm, B.Cu at (178.1, 145.3)
- added TP12: ~, TestPoint:TestPoint_Pad_D1.0mm, B.Cu at (182.6, 147.2)
- added TP13: ~, TestPoint:TestPoint_Pad_D1.0mm, B.Cu at (171.2, 143.8)
- added TP15: ~, TestPoint:TestPoint_Pad_D1.0mm, B.Cu at (174.2, 143.8)
- added TP7: ~, TestPoint:TestPoint_Pad_D1.0mm, B.Cu at (172.7, 143.8)
- added TP9: ~, TestPoint:TestPoint_Pad_D1.0mm, B.Cu at (178.1, 143.8)
- added U20: MAX10M04, Package_QFP:EQFP-144-1EP_20x20mm_P0.5mm_EP5x5mm_ThermalVias, B.Cu at (177.2, 129.5)
- added U22: LM809, Package_TO_SOT_SMD:SOT-23, B.Cu at (169.7, 146.3)
- added U24: TLV74318, Package_TO_SOT_SMD:SOT-23-5, F.Cu at (195.3, 128.0)
- added U25: S80KS2563GABHV020, myspace pcb:FBGA-24_6mmx8mm_Layout5x5_P1.00mm, B.Cu at (194.3, 124.9)
- added X2: ASE-48MHz, Oscillator:Oscillator_SMD_Abracon_ASV-4Pin_7.0x5.1mm_HandSoldering, F.Cu at (185.2, 130.5)
- J4: value Jack -> Jack(Red)
- J7: value Jack -> Jack(Black)
- Q2: value 2N3904 -> MMBT3904
- R26, R55: value 0 -> 0R
- U19, U9: value ~ -> XS-LCC-01
- moved J1 0.14 mm to (159.6, 111.8)
- moved J2 0.14 mm to (159.6, 149.9)
Routing:
- net +3.3V: track 131.5 -> 286.8 mm, vias 32 -> 62
- net /launch_n: track 99.8 -> 238.4 mm, vias 2 -> 3
- net /cont_led: track 123.9 -> 237.3 mm, vias 2 -> 3
- net /osc: track 87.8 -> 187.2 mm, vias 3 -> 5
- net /charge: track 118.8 -> 210.9 mm, vias 3 -> 4
- net /reset_n: track 103.8 -> 195.0 mm, vias 3 -> 4
- net /sclk: track 74.0 -> 157.0 mm, vias 3 -> 4
- net /cs: track 81.1 -> 162.8 mm, vias 3 -> 4
- net /arm_led: track 137.1 -> 218.1 mm, vias 2 -> 3
- net /dataB1: track 65.7 -> 145.6 mm, vias 2 -> 3
- net /dataA1: track 62.4 -> 141.4 mm, vias 2 -> 3
- net /dataA0: track 64.4 -> 142.3 mm, vias 2 -> 3
- net /dataB0: track 63.8 -> 141.5 mm, vias 2 -> 3
- net /pwm: track 128.0 -> 193.9 mm
- net /dump: track 108.7 -> 171.7 mm
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- added copper zone on F.Cu, net +1V8
- added copper zone on In2.Cu, net +1V8
- added copper zone on B.Cu, net GND
- removed copper zone on In3.Cu, net GND
Other:
- outline, holes or cut-outs redrawn
- board text added: "XS-LCC-01-DB01.2"
- board text removed: "XS-LCC-01-DB00.1"
