File: dev_board.kicad_sch (KiCad schematic)
At the start: 225 parts, among them J1 Conn_02x13_Odd_Even, J2 Conn_02x13_Odd_Even, J4 Jack, J5 Conn_01x06, J7 Jack, J9 Barrel_Jack, Q1 STR2P3LLH6(Pfet), Q10 MMBT3904, Q2 2N3904, Q3 MMBT3904, Q4 IPD60R145, Q5 IRLML0060TRPBF, Q6 IPD60R145, Q9 MMBT3904, SW1 SW_SPST, SW10 LAUNCH, SW3 ARM, U1 LT3420, U10 AMC3330, U11 AT25xxx, U12 TLV74318, U13 LM809, U14 AMC3302, U17 AD7352, U18 IR2127, U2 TLV74318, U23 TLV74325, U3 AD7352, U4 TLV74325, U5 LMO78_03-1.0, U6 4945, U7 MCP1416, U8 AMC3330, X1 ASE-48MHz

Commit message: Closer to tapeout, Digikey BOM added
Parts:
- C29, C30, C38, C39, C54, C55, C56, C57: DPN 399-C0603C102K3RAC7867CT-ND -> 399-C0603C222K3RAC7867CT-ND
- D1: DPN (none) -> BAV99LT1GOSCT-ND
- D5: DPN GSD2004S-E3-08CT-N -> GSD2004S-E3-08CT-ND
- GD1: DPN (none) -> F11278CT-ND
- J1, J2: DPN (none) -> ESW-113-12-T-D-ND
- J4: value Jack -> Jack(Red); DPN (none) -> BKCT3151-2-ND
- J5: DPN (none) -> 952-1922-ND
- J7: value Jack -> Jack(Black); DPN (none) -> BKCT3151-0-ND
- L1: DPN M8893-ND -> 595-1735-ND
- PS1: DPN (none) -> 945-1209-ND
- Q10, Q3, Q9: value MMBT3904 -> 2N3904; DPN (none) -> 4530-MMBT3904CT-ND
- R11, R4: DPN P1.00KHCT-ND -> P10.0KHCT-ND
- R25: DPN 541-MCT0603MD2004BP500CT-ND -> 10-ERA-3VRW1002VCT-ND
- R26: value 0 -> 0R; DPN 541-MCT0603MD2004BP500CT-ND -> P0.0GCT-ND
- R55: value 0 -> 0R; DPN P1.00KHCT-ND -> P0.0GCT-ND
- U11: DPN (none) -> 1695-AT25EU0011A-SSHN-TCT-ND
- U19, U9: value ~ -> XS-LCC-01
- U7: DPN (none) -> MCP1416T-E/OTCT-ND
Connections:
- net +1V1: no longer J1.3 (Pin_3)
- no-connect marks 3 -> 4

Commit message: Tapeout v01.2
Parts:
- added C100, C101, C102, C103, C105, C106, C108, C109, C110, C116, C119, C120, C121, C122, C123, C124, C127, C130, C131, C139, C140, C142, C143, C144, C90, C92, C93, C94, C96, C97, C99: 0.1u, Capacitor_SMD:C_0603_1608Metric, symbol Device:C_Small
- added C104, C115, C125, C126, C141, C91, C98: 1u, Capacitor_SMD:C_0603_1608Metric, symbol Device:C_Small
- added C51, C52, C58: 4.7u, Capacitor_SMD:C_1206_3216Metric, symbol Device:C_Small
- added D10, D11, D12, D13, D14, D15, D3, D8: Yel, LED_SMD:LED_0603_1608Metric, symbol Device:LED
- added D16: BAV99, Package_TO_SOT_SMD:SOT-23, symbol Diode:BAV99
- added FB2, FB3, FB4, FB8: Ferrite, Inductor_SMD:L_0603_1608Metric, symbol Device:FerriteBead_Small
- added J10, J14: Conn_02x05_Odd_Even, Connector_PinHeader_2.54mm:PinHeader_2x05_P2.54mm_Vertical, symbol Connector_Generic:Conn_02x05_Odd_Even
- added J12: HDMI_D_1.4, Connector_HDMI:HDMI_A_Amphenol_10029449-x01xLF_Horizontal, symbol Connector:HDMI_A
- added J3, J6: Conn_02x13_Odd_Even, Connector_PinSocket_2.54mm:PinSocket_2x13_P2.54mm_Vertical, symbol Connector_Generic:Conn_02x13_Odd_Even
- added LS2: Speaker, Buzzer_Beeper:PUIAudio_SMT_0825_S_4_R, symbol Device:Speaker
- added Q7: MMBT3904, Package_TO_SOT_SMD:SOT-23, symbol Transistor_BJT:MMBT3904
- added R101, R74, R75, R76, R78: 10K, Resistor_SMD:R_0603_1608Metric, symbol Device:R
- added R56, R84, R90, R97: 0R, Resistor_SMD:R_0603_1608Metric, symbol Device:R
- added R57, R58, R59, R60, R65, R66, R71, R72, R73, R77: 1K, Resistor_SMD:R_0603_1608Metric, symbol Device:R
- added R86, R87, R91: 22R, Resistor_SMD:R_0603_1608Metric, symbol Device:R
- added R88: DNI, Resistor_SMD:R_0603_1608Metric, symbol Device:R
- added SW12: SW_DIP_x03, Button_Switch_SMD:SW_DIP_SPSTx03_Slide_Omron_A6S-310x_W8.9mm_P2.54mm, symbol Switch:SW_DIP_x03
- added SW2: LAUNCH, myspace pcb:SW_SPST_HP03, symbol Switch:SW_Push
- added TP10, TP11, TP12, TP15, TP9: ~, TestPoint:TestPoint_Pad_D1.5mm, symbol Connector:TestPoint
- added TP13, TP7: ~, TestPoint:TestPoint_Pad_D1.0mm, symbol Connector:TestPoint
- added U20: MAX10M04, Package_QFP:EQFP-144-1EP_20x20mm_P0.5mm_EP8.93x8.7mm_ThermalVias, symbol myspace:MAX10_FPGA_M08_LQFP144_
- added U22: LM809, Package_TO_SOT_SMD:SOT-23, symbol Power_Supervisor:LM809
- added U24: TLV74318, Package_TO_SOT_SMD:SOT-23-5, symbol myspace:TLV74325_SOT23-5
- added U25: S80KS2563GABHV020, myspace pcb:FBGA-24_6mmx8mm_Layout5x5_P1.00mm, symbol myspace:S8KS256
- added X2: ASE-48MHz, Oscillator:Oscillator_SMD_Abracon_ASV-4Pin_7.0x5.1mm_HandSoldering, symbol Oscillator:ASE-xxxMHz
- C24, C25: DPN 1572-1041-ND -> 400BXW100MEFR18X25
- J1, J2: footprint (none) -> Connector_PinSocket_2.54mm:PinSocket_2x13_P2.54mm_Vertical
- Q10, Q2, Q3, Q9: value 2N3904 -> MMBT3904
- Q5: DPN 448-IPD60R145CFD7ATMA1CT-ND -> IRLML0060TRPBFCT-ND
- R1, R2, R29: DPN P100KHCT-ND -> RMCF0603FT100KCT-ND
- R10, R11, R12, R14, R4, R43, R53, R6, R7, R83, R9, R98: DPN P10.0KHCT-ND -> 311-10.0KHRCT-ND
- R102: DPN 541-3275-1-ND -> 846-GMR320HJAAFD5L00CT-ND
- R27: DPN 10-ERA-3VRW1002VCT-ND -> 10-ERA-3VRW1001VCT-ND
- R32, R37, R38, R41, R42, R45: DPN P1.00KHCT-ND -> (none); JLC C319967 -> (none)
- R35, R36, R39, R40, R61, R62, R63, R64: DPN P22.0HCT-ND -> P51.0HCT-ND
- R44: DPN P1.00KHCT-ND -> 311-3.30KHRCT-ND
- SW3: DPN EG2585-ND -> 360-2595-1-ND
- U10, U8: DPN 296-AMC3330QDWERQ1CT-ND -> 296-AMC3330DWE-ND
- U17, U3: DPN 505-AD7352BRUZ-ND -> AD7352YRUZ-ND
Connections:
- net +3.3V: now also C101.1, C103.1, C106.1, C108.1, C109.1, C110.1, C119.1, C120.1, C121.1, C122.1, C123.1, C124.1, C125.1, C139.1, C140.1, C143.1, C144.1, C51.1, C52.1, C58.1, C90.1, C92.1, C93.1, C96.1, C99.1, D10.2 (A), D11.2 (A), D12.2 (A), D13.2 (A), D14.2 (A), D15.2 (A), D16.3 (K), D3.2 (A), D8.2 (A), FB2.1, FB3.1, FB4.1, FB8.1, J3.4 (Pin_4), LS2.1, R101.2, R74.1, R84.1, R90.1, R97.1, U20.1 (VCC_ONE), U20.103 (VCCIO6), U20.108 (VCC_ONE), U20.109 (VCC_ONE), U20.115 (VCC_ONE), U20.128 (VCCIO8), U20.139 (VCCIO8), U20.144 (VCC_ONE), U20.31 (VCCIO2), U20.36 (VCC_ONE), U20.37 (VCC_ONE), U20.40 (VCCIO3), U20.49 (VCCIO3), U20.51 (VCC_ONE), U20.67 (VCCIO4), U20.72 (VCC_ONE), U20.73 (VCC_ONE), U20.9 (VCCIO1A), U20.94 (VCCIO6), U22.3 (VCC), U24.1 (IN), U24.3 (EN), X2.1 (EN), X2.4 (Vdd)
- net GND: now also C100.2, C101.2, C102.2, C103.2, C104.2, C105.2, C106.2, C108.2, C109.2, C110.2, C115.2, C116.2, C119.2, C120.2, C121.2, C122.2, C123.2, C124.2, C125.2, C126.2, C127.2, C130.2, C131.2, C139.2, C140.2, C141.2, C142.2, C143.2, C144.2, C51.2, C52.2, C58.2, C90.2, C91.2, C92.2, C93.2, C94.2, C96.2, C97.2, C98.2, C99.2, J10.10 (Pin_10), J10.2 (Pin_2), J12.11 (CKS), J12.17 (GND), J12.2 (D2S), J12.5 (D1S), J12.8 (D0S), J12.SH, J14.10 (Pin_10), J14.3 (Pin_3), J3.1 (Pin_1), J3.11 (Pin_11), J3.13 (Pin_13), J3.15 (Pin_15), J3.17 (Pin_17), J3.19 (Pin_19), J3.2 (Pin_2), J3.21 (Pin_21), J3.22 (Pin_22), J3.23 (Pin_23), J3.25 (Pin_25), J3.3 (Pin_3), J3.5 (Pin_5), J3.7 (Pin_7), J3.9 (Pin_9), J6.1 (Pin_1), J6.10 (Pin_10), J6.12 (Pin_12), J6.14 (Pin_14), J6.16 (Pin_16), J6.18 (Pin_18), J6.2 (Pin_2), J6.20 (Pin_20), J6.22 (Pin_22), J6.24 (Pin_24), J6.26 (Pin_26), J6.4 (Pin_4), J6.6 (Pin_6), J6.8 (Pin_8), Q7.2 (E), R77.2, SW12.1, SW12.2, SW12.3, SW2.1, U20.104 (GND), U20.116 (GND), U20.125 (GND), U20.133 (GND), U20.137 (GND), U20.142 (GND), U20.145 (GND_PAD), U20.4 (REFGDN), U20.42 (GND), U20.53 (GND), U20.63 (GND), U20.68 (GND), U20.83 (GND), U20.95 (GND), U22.1 (GND), U24.2 (GND), U25.B3 (VSS), U25.C1 (VssQ), U25.E5 (VssQ), X2.2 (GND)
- net arm_led: now also J6.25 (Pin_25), U20.132 (IO)
- net charge: now also J3.6 (Pin_6), U20.62 (IO)
- net cont_led: now also J6.5 (Pin_5), U20.135 (IO)
- net cs: now also J6.21 (Pin_21), U20.106 (IO)
- net dataA0: now also J6.13 (Pin_13), U20.99 (IO)
- net dataA1: now also J6.17 (Pin_17), U20.102 (IO)
- net dataB0: now also J6.15 (Pin_15), U20.100 (IO)
- net dataB1: now also J6.19 (Pin_19), U20.105 (IO)
- net dump: now also J6.9 (Pin_9), U20.66 (IO)
- net launch_n: now also J6.7 (Pin_7), R91.1, U20.124 (IO)
- net mute_n: now also J3.18 (Pin_18), R56.2
- net osc: now also J3.16 (Pin_16), R86.1, U20.29 (CLK1P)
- net pwm: now also J6.23 (Pin_23), U20.65 (IO)
- net reset_n: now also J3.24 (Pin_24), R87.1, R88.1, U20.28 (CLK1N)
- net sclk: now also J6.11 (Pin_11), U20.101 (IO)
- net speaker: now also J3.20 (Pin_20), R73.1, U20.140 (IO)
- new net: D14.1 (K), R71.1
- new net: D3.1 (K), R57.1
- new net: R101.1, U20.129 (NCONFIG)
- new net: R87.2, U22.2 (~{RESET})
- new net: D15.1 (K), R72.1
- new net: D13.1 (K), R66.1
- new net: R86.2, X2.3 (OUT)
- new net: D16.1 (K), LS2.2, Q7.3 (C)
- new net: D11.1 (K), R60.1
- new net: Q7.1 (B), R73.2
- new net: R74.2, R91.2, SW2.2
- new net: D10.1 (K), R59.1
- new net: D8.1 (K), R58.1
- new net: D12.1 (K), R65.1
- new net +1V8: C126.1, C127.1, C130.1, C131.1, U20.82 (VCCIO5), U24.5 (OUT), U25.B1 (nCK), U25.B4 (VCC), U25.D1 (VccQ), U25.E4 (VccQ)
- new net +3.3VA: C100.1, C102.1, C104.1, C105.1, C91.1, C94.1, C97.1, C98.1, FB2.2, FB3.2, FB4.2, FB8.2, U20.107 (VCCA), U20.143 (VCCA), U20.2 (VCCA), U20.34 (VCCA), U20.35 (VCCA), U20.5 (ADC_VREF), U20.71 (VCCA)
- new net VCCIO1B: C115.1, C116.1, J10.4 (Pin_4), R75.1, R76.1, R78.1, R84.2, U20.23 (VCCIO1B)
- new net ain_1: R57.2, U20.14 (ADC1IN8)
- new net ain_2: R58.2, U20.13 (ADC1IN7)
- new net ain_3: R59.2, U20.12 (ADC1IN6)
- new net ain_4: R60.2, U20.11 (ADC1IN5)
- new net ain_5: R65.2, U20.10 (ADC1IN4)
- new net ain_6: R66.2, U20.8 (ADC1IN3)
- new net ain_7: R71.2, U20.7 (ADC1IN2)
- new net ain_8: R72.2, U20.6 (ADC1IN1)
- new net arm: R97.2, TP12.1, U20.120 (IO)
- new net bootsel: TP9.1, U20.126 (BOOTSEL)
- new net conf_done: TP13.1, U20.138 (CONF_DONE)
- new net crc: TP15.1, U20.134 (CRC_ERR)
- new net devclrn: R88.2, TP11.1, U20.121 (DEVCLRN)
- new net devoe: TP10.1, U20.122 (DEVOE)
- new net dio0: J14.1 (Pin_1), U20.118 (IO)
- new net dio1: J14.2 (Pin_2), U20.119 (IO)
- new net dio2: J14.5 (Pin_5), U20.113 (IO)
- new net dio3: J14.6 (Pin_6), U20.114 (IO)
- new net dio4: J14.7 (Pin_7), U20.111 (IO)
- new net dio5: J14.8 (Pin_8), U20.112 (VREFB7N)
- new net dio6: J14.9 (Pin_9), U20.110 (IO)
- new net hdmi_ck+: J12.10 (CK+), U20.52 (IO)
- new net hdmi_ck-: J12.12 (CK-), U20.50 (IO)
- new net hdmi_d0+: J12.7 (D0+), U20.56 (IO)
- new net hdmi_d0-: J12.9 (D0-), U20.55 (IO)
- new net hdmi_d1+: J12.4 (D1+), U20.58 (IO)
- new net hdmi_d1-: J12.6 (D1-), U20.57 (IO)
- new net hdmi_d2+: J12.1 (D2+), U20.60 (IO)
- new net hdmi_d2-: J12.3 (D2-), U20.59 (IO)
- new net iset0: R56.1, SW12.6, U20.127 (IO)
- new net iset1: SW12.5, U20.130 (IO)
- new net iset2: SW12.4, U20.131 (IO)
- new net jtagen: J10.8 (Pin_8), R78.2, U20.15 (JTAGEN)
- new net nstatus: TP7.1, U20.136 (NSTATUS)
- new net spi_clk: U20.87 (IO), U25.B2 (CK)
- new net spi_cs: U20.81 (IO), U25.A3 (nCS)
- new net spi_d0: U20.78 (IO), U25.D3 (DQ0)
- new net spi_d1: U20.85 (IO), U25.D2 (DQ1)
- new net spi_d2: U20.75 (IO), U25.C4 (DQ2)
- new net spi_d3: U20.77 (IO), U25.D4 (DQ3)
- new net spi_d4: U20.76 (IO), U25.D5 (DQ4)
- new net spi_d5: U20.79 (IO), U25.E3 (DQ5)
- new net spi_d6: U20.84 (IO), U25.E2 (DQ6)
- new net spi_d7: U20.86 (IO), U25.E1 (DQ7)
- new net spi_ds: U20.74 (IO), U25.C3 (RWDS)
- new net spi_nrst: U20.80 (VREFB5N), U25.A4 (nRST)
- new net tck: J10.1 (Pin_1), R77.1, U20.18 (TCK)
- new net tdi: J10.9 (Pin_9), R75.2, U20.19 (TDI)
- new net tdo: J10.3 (Pin_3), U20.20 (TDO)
- new net tms: J10.5 (Pin_5), R76.2, U20.16 (TMS)
- new net vccio7: C141.1, C142.1, J14.4 (Pin_4), R90.2, U20.117 (VCCIO7)
- no-connect marks 4 -> 56
Other:
- note added: "*clk+*"
- note added: "*clk-*"
- note added: "*done*"
- note added: "*rx*"
- note added: "*tx*"
- note added: "2x HDMI Video Out"
- note added: "32MB Capture Buffer Octal xSPI 400 MB/s"
- note added: "4x 3msps 12bit ADC Interface"
- note added: "Analog Expansion"
- note added: "Clock & Reset"
- note added: "Development Support (Optional)"
- note added: "Digital I/O"
- note added: "Emulation and Monitor Probe"
- note added: "Emulator Connector"
- note added: "Energy Storage and Control"
- note added: "Evaluation Probe"
- note added: "FPGA Config"
- note added: "FPGA Power"
- note added: "Front Panel"
- note added: "Front Panel and Config"
- note added: "High Voltage Control"
- note added: "Instrumentation"
- note added: "Launch Control Chip"
- note added: "Launch Controller"
- note added: "XS LCC"
- note removed: "FPanel"
- note removed: "Pwr Ctl"
- note removed: "Quad ADC"
- note removed: "SPI"
- note removed: "Sampling ADCs simultaneous 4ch 12bit 3mhz isolated zero latency"
- note removed: "System"
- note removed: "XS"
- moved on the sheet: BT1, BT2, C1, C10, C11, C12, C128, C129, C13, C132, C133, C134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
